File: schematics/kicad_schematics/bearboard.sch (KiCad schematic (older format))
At the start: 86 parts, among them P1 KOBICONN, P10 CONN_4, P11 CONN_10X2, P2 CONN_10X2, P3 CONN_10X2, P4 CONN_10X2, P5 CONN_10X2, P6 CONN_10X2, P7 CONN_10X2, P8 CONN_10X2, P9 CONN_7, SW1 SW_PUSH, SW5 SWITCH, SW6 SWITCH, U1 VBAT, U14 SD_CARD, U2 STM32F103, U3 TACT-SKQU, U4 EMA406GPS, X1 8-16MHz, X2 32.768KHz, X3 ARDUINOSHIELD

Commit message: added datasheets and modified schematic components for new dip switches
Parts:
- removed SW1: SW_PUSH, symbol SW_PUSH
- removed SW5, SW6: SWITCH, symbol SWITCH
- added SW5: SW_TACT, symbol SW_TACT
- added SW6: DIP_SPDT_2, symbol DIP_SPDT_2
Connections:
- wire segments 539 -> 542
Other:
- moved on the sheet: R2

Commit message: Updated schematics removing spaces
Parts:
- added C53, C54, C55, C56, C57, C58, C59, C60, C61, C62, C63: 100nF, SM0805, symbol C
- SW5: footprint (none) -> tactileButtonTL3315
- SW6: footprint (none) -> SPDT-DIP-204-122
- U14: footprint (none) -> SD-Card-Holder-145
- X1: value 8-16MHz -> 8MHz; footprint (none) -> 8Mz-Crystal
Connections:
- net 3V3: now also C53.1, C54.1, C55.1, C56.1, C57.1, C58.1, C59.1, C60.1, C61.1, C62.1, C63.1
- net GND: now also C53.2, C54.2, C55.2, C56.2, C57.2, C58.2, C59.2, C60.2, C61.2, C62.2, C63.2
- net VDDA: no longer C2.1, L1.1
- new net: C2.1, L1.1
Other:
- note added: "POWER SUPPLY DECOUPLERS"

Commit message: made some usb changes
Parts:
- U14: footprint SD-Card-Holder-145 -> (none)
Changed lines of the file:
@@
-EESchema Schematic File Version 2  date Sun 14 Mar 2010 02:53:54 PM EDT
+EESchema Schematic File Version 2  date Sun 14 Mar 2010 03:28:34 PM EDT
 LIBS:power
 LIBS:device
@@
 Comment4 ""
 $EndDescr
+$Comp
+L SD_CARD U14
+U 1 1 4B9D33B5
+P 20400 10450
+F 0 "U14" H 20250 11350 60  0000 C CNN
+F 1 "SD_CARD" H 20400 9550 60  0000 C CNN
+	1    20400 10450
+	1    0    0    -1
+$EndComp
 Wire Bus Line
 	18250 14500 18250 12300
@@
 Wire Wire Line
 	19700 10450 19900 10450
-Connection ~ 19700 11350
 Connection ~ 18750 10750
 Wire Wire Line
@@
 	18500 9500 18500 10900
 Connection ~ 18500 10900
-Wire Wire Line
-	19900 11350 19700 11350
 Connection ~ 19700 10450
 Wire Wire Line
@@
 	-1   0    0    1
 $EndComp
-$Comp
-L SD_CARD U14
-U 1 1 4B981B1A
-P 20400 10450
-F 0 "U14" H 20250 11350 60  0000 C CNN
-F 1 "SD_CARD" H 20400 9400 60  0000 C CNN
-F 2 "SD-Card-Holder-145" H 20400 10450 60  0001 C CNN
-	1    20400 10450
-	1    0    0    -1
-$EndComp
 Text Label 7150 6250 0    60   ~ 0

Commit message: modified pinout on em406, update schematic, and modified pinout on S08 and SSOT6
Parts:
- D1, D2, D3: footprint SC-59 -> DO-124AB-DIODE
- U14: footprint (none) -> SD-Card-Holder-145
- U4: footprint EM406 -> (none)
Changed lines of the file:
@@
-EESchema Schematic File Version 2  date Sun 14 Mar 2010 03:28:34 PM EDT
+EESchema Schematic File Version 2  date Sun 14 Mar 2010 03:55:01 PM EDT
 LIBS:power
 LIBS:device
@@
 $EndDescr
 $Comp
+L EMA406GPS U4
+U 1 1 4B9D3AA3
+P 13700 13000
+F 0 "U4" H 13750 13450 60  0000 C CNN
+F 1 "EMA406GPS" H 13950 12650 60  0000 C CNN
+	1    13700 13000
+	1    0    0    -1
+$EndComp
+$Comp
 L SD_CARD U14
 U 1 1 4B9D33B5
@@
 F 0 "U14" H 20250 11350 60  0000 C CNN
 F 1 "SD_CARD" H 20400 9550 60  0000 C CNN
+F 2 "SD-Card-Holder-145" H 20400 10450 60  0001 C CNN
 	1    20400 10450
 	1    0    0    -1
@@
 F 0 "D1" H 2900 1150 40  0000 C CNN
 F 1 "DIODESCH" H 2900 950 40  0000 C CNN
-F 2 "SC-59" H 2900 1050 60  0001 C CNN
+F 2 "DO-124AB-DIODE" H 2900 1050 60  0001 C CNN
 	1    2900 1050
 	1    0    0    -1
@@
 $EndComp
 NoConn ~ 13400 12700
-$Comp
-L EMA406GPS U4
-U 1 1 4B91D30F
-P 13700 13000
-F 0 "U4" H 13750 13450 60  0000 C CNN
-F 1 "EMA406GPS" H 13950 12650 60  0000 C CNN
-F 2 "EM406" H 13700 13000 60  0001 C CNN
-	1    13700 13000
-	1    0    0    -1
-$EndComp
 Text Label 15950 14250 0    60   ~ 0
 USART2_CTS
@@
 F 0 "D2" H 2900 1450 40  0000 C CNN
 F 1 "DIODESCH" H 2900 1250 40  0000 C CNN
-F 2 "SC-59" H 2900 1350 60  0001 C CNN
+F 2 "DO-124AB-DIODE" H 2900 1350 60  0001 C CNN
 	1    2900 1350
 	1    0    0    -1
@@
 F 0 "D3" H 2900 1750 40  0000 C CNN
 F 1 "DIODESCH" H 2900 1550 40  0000 C CNN
-F 2 "SC-59" H 2900 1650 60  0001 C CNN
+F 2 "DO-124AB-DIODE" H 2900 1650 60  0001 C CNN
 	1    2900 1650
 	1    0    0    -1

Commit message: started PCB schematic
Parts:
- U4: footprint (none) -> EM406
Changed lines of the file:
@@
-EESchema Schematic File Version 2  date Mon 15 Mar 2010 01:44:05 PM EDT
+EESchema Schematic File Version 2  date Mon 15 Mar 2010 09:49:52 PM EDT
 LIBS:power
 LIBS:device
@@
 Sheet 1 5
 Title "BearBoard STM32F103"
-Date "15 mar 2010"
+Date "16 mar 2010"
 Rev "0"
 Comp "University of Maine"
@@
 F 0 "U4" H 13750 13450 60  0000 C CNN
 F 1 "EMA406GPS" H 13950 12650 60  0000 C CNN
+F 2 "EM406" H 13700 13000 60  0001 C CNN
 	1    13700 13000
 	1    0    0    -1
@@
 POWER SUPPLY DECOUPLERS
 $Comp
-L GND #PWR01
+L GND #PWR28
 U 1 1 4B9D17C9
 P 19400 13400
-F 0 "#PWR01" H 19400 13400 30  0001 C CNN
+F 0 "#PWR28" H 19400 13400 30  0001 C CNN
 F 1 "GND" H 19400 13330 30  0001 C CNN
 	1    19400 13400
@@
 3V3
 $Comp
-L GND #PWR02
+L GND #PWR29
 U 1 1 4B9D1705
 P 19400 14400
-F 0 "#PWR02" H 19400 14400 30  0001 C CNN
+F 0 "#PWR29" H 19400 14400 30  0001 C CNN
 F 1 "GND" H 19400 14330 30  0001 C CNN
 	1    19400 14400
@@
 USB5V
 $Comp
-L 3V3 #PWR03
+L 3V3 #PWR31
 U 1 1 4B981769
 P 19800 8800
-F 0 "#PWR03" H 19800 8900 40  0001 C CNN
+F 0 "#PWR31" H 19800 8900 40  0001 C CNN
 F 1 "3V3" H 19800 8949 40  0000 C CNN
 	1    19800 8800
@@
 BOOT1
 $Comp
-L GND #PWR04
+L GND #PWR2
 U 1 1 4B980614
 P 750 3350
-F 0 "#PWR04" H 750 3350 30  0001 C CNN
+F 0 "#PWR2" H 750 3350 30  0001 C CNN
 F 1 "GND" H 750 3280 30  0001 C CNN
 	1    750  3350
@@
 $EndComp
 $Comp
-L 3V3 #PWR05
+L 3V3 #PWR1
 U 1 1 4B9805B2
 P 750 2650
-F 0 "#PWR05" H 750 2750 40  0001 C CNN
+F 0 "#PWR1" H 750 2750 40  0001 C CNN
 F 1 "3V3" H 750 2799 40  0000 C CNN
 	1    750  2650
@@
 POWER SUPPLY
 $Comp
-L 3V3 #PWR06
+L 3V3 #PWR14
 U 1 1 4B97F193
 P 5050 1250
-F 0 "#PWR06" H 5050 1350 40  0001 C CNN
+F 0 "#PWR14" H 5050 1350 40  0001 C CNN
 F 1 "3V3" H 5050 1399 40  0000 C CNN
 	1    5050 1250
@@
 VBAT
 $Comp
-L 3V3 #PWR07
+L 3V3 #PWR9
 U 1 1 4B97F11B
 P 1700 6150
-F 0 "#PWR07" H 1700 6250 40  0001 C CNN
+F 0 "#PWR9" H 1700 6250 40  0001 C CNN
 F 1 "3V3" H 1700 6299 40  0000 C CNN
 	1    1700 6150
@@
 JOY_UP
 $Comp
-L 3V3 #PWR08
+L 3V3 #PWR25
 U 1 1 4B97EDF8
 P 19000 6100
-F 0 "#PWR08" H 19000 6200 40  0001 C CNN
+F 0 "#PWR25" H 19000 6200 40  0001 C CNN
 F 1 "3V3" H 19000 6249 40  0000 C CNN
 	1    19000 6100
@@
 $EndComp
 $Comp
-L GND #PWR09
+L GND #PWR32
 U 1 1 4B97EDCC
 P 19850 7750
-F 0 "#PWR09" H 19850 7750 30  0001 C CNN
+F 0 "#PWR32" H 19850 7750 30  0001 C CNN
 F 1 "GND" H 19850 7680 30  0001 C CNN
 	1    19850 7750
@@
 $EndComp
 $Comp
-L GND #PWR010
+L GND #PWR26
 U 1 1 4B97D0B2
 P 19000 8250
-F 0 "#PWR010" H 19000 8250 30  0001 C CNN
+F 0 "#PWR26" H 19000 8250 30  0001 C CNN
 F 1 "GND" H 19000 8180 30  0001 C CNN
 	1    19000 8250
@@
 USART2_TX
 $Comp
-L GND #PWR011
+L GND #PWR16
 U 1 1 4B97C2CE
 P 5950 6150
-F 0 "#PWR011" H 5950 6150 30  0001 C CNN
+F 0 "#PWR16" H 5950 6150 30  0001 C CNN
 F 1 "GND" H 5950 6080 30  0001 C CNN
 	1    5950 6150
@@
 $EndComp
 $Comp
-L GND #PWR012
+L GND #PWR7
 U 1 1 4B97BC68
 P 1500 1500
-F 0 "#PWR012" H 1500 1500 30  0001 C CNN
+F 0 "#PWR7" H 1500 1500 30  0001 C CNN
 F 1 "GND" H 1500 1430 30  0001 C CNN
 	1    1500 1500
@@
 SD CARD INTERFACE
 $Comp
-L GND #PWR013
+L GND #PWR20
 U 1 1 4B91D59F
 P 11950 13550
-F 0 "#PWR013" H 11950 13550 30  0001 C CNN
+F 0 "#PWR20" H 11950 13550 30  0001 C CNN
 F 1 "GND" H 11950 13480 30  0001 C CNN
 	1    11950 13550
@@
 $EndComp
 $Comp
-L GND #PWR014
+L GND #PWR21
 U 1 1 4B91D596
 P 13250 13300
-F 0 "#PWR014" H 13250 13300 30  0001 C CNN
+F 0 "#PWR21" H 13250 13300 30  0001 C CNN
 F 1 "GND" H 13250 13230 30  0001 C CNN
 	1    13250 13300
@@
 $EndComp
 $Comp
-L 3V3 #PWR015
+L 3V3 #PWR23
 U 1 1 4B918558
 P 18600 4250
-F 0 "#PWR015" H 18600 4350 40  0001 C CNN
+F 0 "#PWR23" H 18600 4350 40  0001 C CNN
 F 1 "3V3" H 18600 4399 40  0000 C CNN
 	1    18600 4250
@@
 5V0
 $Comp
-L GND #PWR016
+L GND #PWR22
 U 1 1 4B906F37
 P 13600 10900
-F 0 "#PWR016" H 13600 10900 30  0001 C CNN
+F 0 "#PWR22" H 13600 10900 30  0001 C CNN
 F 1 "GND" H 13600 10830 30  0001 C CNN
 	1    13600 10900
@@
 VDDA
 $Comp
-L GND #PWR017
+L GND #PWR6
 U 1 1 4B906833
 P 1400 7850
-F 0 "#PWR017" H 1400 7850 30  0001 C CNN
+F 0 "#PWR6" H 1400 7850 30  0001 C CNN
 F 1 "GND" H 1400 7780 30  0001 C CNN
 	1    1400 7850
@@
 $EndComp
 $Comp
-L 3V3 #PWR018
+L 3V3 #PWR4
 U 1 1 4B906827
 P 750 7300
-F 0 "#PWR018" H 750 7400 40  0001 C CNN
+F 0 "#PWR4" H 750 7400 40  0001 C CNN
 F 1 "3V3" H 750 7449 40  0000 C CNN
 	1    750  7300
@@
 $EndComp
 $Comp
-L GND #PWR019
+L GND #PWR11
 U 1 1 4B906768
 P 2800 8250
-F 0 "#PWR019" H 2800 8250 30  0001 C CNN
+F 0 "#PWR11" H 2800 8250 30  0001 C CNN
 F 1 "GND" H 2800 8180 30  0001 C CNN
 	1    2800 8250
@@
 $EndComp
 $Comp
-L GND #PWR020
+L GND #PWR10
 U 1 1 4B906595
 P 1700 6700
-F 0 "#PWR020" H 1700 6700 30  0001 C CNN
+F 0 "#PWR10" H 1700 6700 30  0001 C CNN
 F 1 "GND" H 1700 6630 30  0001 C CNN
 	1    1700 6700
@@
 $EndComp
 $Comp
-L 3V3 #PWR021
+L 3V3 #PWR19
 U 1 1 4B906233
 P 9300 12950
-F 0 "#PWR021" H 9300 13050 40  0001 C CNN
+F 0 "#PWR19" H 9300 13050 40  0001 C CNN
 F 1 "3V3" H 9300 13099 40  0000 C CNN
 	1    9300 12950
@@
 $EndComp
 $Comp
-L 3V3 #PWR022
+L 3V3 #PWR8
 U 1 1 4B905C37
 P 1550 4350
-F 0 "#PWR022" H 1550 4450 40  0001 C CNN
+F 0 "#PWR8" H 1550 4450 40  0001 C CNN
 F 1 "3V3" H 1550 4499 40  0000 C CNN
 	1    1550 4350
@@
 $EndComp
 $Comp
-L 3V3 #PWR023
+L 3V3 #PWR17
 U 1 1 4B9034AD
 P 8100 14100
-F 0 "#PWR023" H 8100 14200 40  0001 C CNN
+F 0 "#PWR17" H 8100 14200 40  0001 C CNN
 F 1 "3V3" H 8100 14249 40  0000 C CNN
 	1    8100 14100
@@
 TMS/SWDIO
 $Comp
-L GND #PWR024
+L GND #PWR18
 U 1 1 4B903530
 P 8100 15950
-F 0 "#PWR024" H 8100 15950 30  0001 C CNN
+F 0 "#PWR18" H 8100 15950 30  0001 C CNN
 F 1 "GND" H 8100 15880 30  0001 C CNN
 	1    8100 15950
@@
 GND
 $Comp
-L GND #PWR025
+L GND #PWR3
 U 1 1 4B9032D4
 P 750 5450
-F 0 "#PWR025" H 750 5450 30  0001 C CNN
+F 0 "#PWR3" H 750 5450 30  0001 C CNN
 F 1 "GND" H 750 5380 30  0001 C CNN
 	1    750  5450
@@
 RESET#
 $Comp
-L 3V3 #PWR026
+L 3V3 #PWR24
 U 1 1 4B903136
 P 18650 1750
-F 0 "#PWR026" H 18650 1850 40  0001 C CNN
+F 0 "#PWR24" H 18650 1850 40  0001 C CNN
 F 1 "3V3" H 18650 1899 40  0000 C CNN
 	1    18650 1750
@@
 FSMC_NOE
 $Comp
-L GND #PWR027
+L GND #PWR13
 U 1 1 4B9001FC
 P 3500 1700
-F 0 "#PWR027" H 3500 1700 30  0001 C CNN
+F 0 "#PWR13" H 3500 1700 30  0001 C CNN
 F 1 "GND" H 3500 1630 30  0001 C CNN
 	1    3500 1700
@@
 $EndComp
 $Comp
-L +5V #PWR028
+L +5V #PWR15
 U 1 1 4B9001CE
 P 5300 1250
-F 0 "#PWR028" H 5300 1340 20  0001 C CNN
+F 0 "#PWR15" H 5300 1340 20  0001 C CNN
 F 1 "+5V" H 5300 1340 30  0000 C CNN
 	1    5300 1250
@@
 $EndComp
 $Comp
-L GND #PWR029
+L GND #PWR12
 U 1 1 4B7EA0B9
 P 3000 10700
-F 0 "#PWR029" H 3000 10700 30  0001 C CNN
+F 0 "#PWR12" H 3000 10700 30  0001 C CNN
 F 1 "GND" H 3000 10630 30  0001 C CNN
 	1    3000 10700
@@
 $EndComp
 $Comp
-L GND #PWR030
+L GND #PWR5
 U 1 1 4B7E9BE8
 P 1350 10750
-F 0 "#PWR030" H 1350 10750 30  0001 C CNN
+F 0 "#PWR5" H 1350 10750 30  0001 C CNN
 F 1 "GND" H 1350 10680 30  0001 C CNN
 	1    1350 10750
@@
 SD_DAT3
 $Comp
-L GND #PWR031
+L GND #PWR30
 U 1 1 4B7E2670
 P 19700 11600
-F 0 "#PWR031" H 19700 11600 30  0001 C CNN
+F 0 "#PWR30" H 19700 11600 30  0001 C CNN
 F 1 "GND" H 19700 11530 30  0001 C CNN
 	1    19700 11600
@@
 $EndComp
 $Comp
-L 3V3 #PWR032
+L 3V3 #PWR27
 U 1 1 4B7E255C
 P 19000 8800
-F 0 "#PWR032" H 19000 8900 40  0001 C CNN
+F 0 "#PWR27" H 19000 8900 40  0001 C CNN
 F 1 "3V3" H 19000 8949 40  0000 C CNN
 	1    19000 8800

Commit message: Modified power libraries. Now using custom power.lib. This is important Removed outdated crystal libaries Changed some caps to 0603 mounts started PCB layout
Parts:
- C1, C10, C11, C12, C13, C2, C3, C4, C5, C53, C54, C55, C56, C57, C58, C59, C6, C60, C61, C62, C63, C7, C8, C9, L1, R1, R10, R11, R12, R13, R14, R15, R16, R17, R18, R19, R2, R20, R21, R22, R23, R24, R25, R26, R27, R28, R29, R3, R30, R31, R32, R33, R34, R35, R36, R37, R38, R4, R5, R6, R7, R70, R71, R8, R9: footprint SM0805 -> SM0805-CUSTOM
- D4, D5, D6, D7: footprint LED-0805 -> LED-0805-CUS
Connections:
- net +5V renamed 5V0
