File: schematics/kicad_schematics/power_supply.sch (KiCad schematic (older format))
At the start: 28 parts, among them Q3 MOSFET_N, Q4 NMOS, U10 LTC3827, U11 LTC1771

Commit message: back annotated footprints into eeschem schematic
Parts:
- C37, C38, C39, C40, C41, C42, C43, C44, C47, C49, R61, R62, R63, R64, R65, R66, R67: footprint (none) -> SM0805
- C45, C46: footprint (none) -> SM1210L
- C48: footprint (none) -> CP10
- U10: footprint (none) -> TSOT-23
- U11: footprint (none) -> MSOP8
Changed lines of the file:
@@
-EESchema Schematic File Version 2  date Wed 10 Mar 2010 08:20:30 PM EST
+EESchema Schematic File Version 2  date Fri 12 Mar 2010 11:31:07 AM EST
 LIBS:power
 LIBS:device
@@
 F 0 "C40" H 2700 4550 50  0000 L CNN
 F 1 "47pF" H 2700 4350 50  0000 L CNN
+F 2 "SM0805" H 2650 4450 60  0001 C CNN
 	1    2650 4450
 	0    1    1    0
@@
 F 0 "C38" H 2450 4800 50  0000 L CNN
 F 1 "1.8nF" H 2450 4600 50  0000 L CNN
+F 2 "SM0805" H 2400 4700 60  0001 C CNN
 	1    2400 4700
 	0    1    1    0
@@
 F 0 "R62" V 3030 4700 50  0000 C CNN
 F 1 "17.4K" V 2950 4700 50  0000 C CNN
+F 2 "SM0805" H 2950 4700 60  0001 C CNN
 	1    2950 4700
 	0    1    1    0
@@
 F 0 "C41" H 3300 5900 50  0000 L CNN
 F 1 "5pF" H 3300 5700 50  0000 L CNN
+F 2 "SM0805" H 3250 5800 60  0001 C CNN
 	1    3250 5800
 	1    0    0    -1
@@
 F 0 "R63" V 3250 5300 50  0000 C CNN
 F 1 "11k 1%" V 3350 5300 50  0000 C CNN
+F 2 "SM0805" H 3250 5300 60  0001 C CNN
 	1    3250 5300
 	0    1    1    0
@@
 F 0 "R65" V 3550 5800 50  0000 C CNN
 F 1 "34.8k 1%" V 3650 5800 50  0000 C CNN
+F 2 "SM0805" H 3550 5800 60  0001 C CNN
 	1    3550 5800
 	1    0    0    -1
@@
 F 0 "C43" H 4350 6100 50  0000 L CNN
 F 1 "1nF" H 4350 5900 50  0000 L CNN
+F 2 "SM0805" H 4300 6000 60  0001 C CNN
 	1    4300 6000
 	1    0    0    -1
@@
 F 0 "C44" H 6000 5050 50  0000 L CNN
 F 1 "10uF" H 6000 4850 50  0000 L CNN
+F 2 "SM0805" H 5950 4950 60  0001 C CNN
 	1    5950 4950
 	1    0    0    -1
@@
 F 0 "C47" H 7000 5850 50  0000 L CNN
 F 1 "10uF" H 7000 5650 50  0000 L CNN
+F 2 "SM0805" H 6950 5750 60  0001 C CNN
 	1    6950 5750
 	1    0    0    -1
@@
 F 0 "C46" H 6650 5850 50  0000 L CNN
 F 1 "100uF" H 6650 5650 50  0000 L CNN
+F 2 "SM1210L" H 6600 5750 60  0001 C CNN
 	1    6600 5750
 	1    0    0    -1
@@
 F 0 "C45" H 6300 5850 50  0000 L CNN
 F 1 "100uF" H 6300 5650 50  0000 L CNN
+F 2 "SM1210L" H 6250 5750 60  0001 C CNN
 	1    6250 5750
 	1    0    0    -1
@@
 F 0 "U10" H 4650 4600 60  0000 C CNN
 F 1 "LTC3827" H 4300 5500 60  0000 C CNN
+F 2 "TSOT-23" H 4300 5050 60  0001 C CNN
 	1    4300 5050
 	1    0    0    -1
@@
 F 0 "C42" H 3450 3600 50  0000 L CNN
 F 1 "5pF" H 3450 3400 50  0000 L CNN
+F 2 "SM0805" H 3400 3500 60  0001 C CNN
 	1    3400 3500
 	0    1    1    0
@@
 F 0 "R66" V 4000 3750 50  0000 C CNN
 F 1 "1M 1%" V 4100 3750 50  0000 C CNN
+F 2 "SM0805" H 4000 3750 60  0001 C CNN
 	1    4000 3750
 	0    1    1    0
@@
 F 0 "R64" V 3400 3750 50  0000 C CNN
 F 1 "1.64M 1%" V 3500 3750 50  0000 C CNN
+F 2 "SM0805" H 3400 3750 60  0001 C CNN
 	1    3400 3750
 	0    1    1    0
@@
 F 0 "C39" H 2650 3650 50  0000 L CNN
 F 1 "220pF" H 2650 3450 50  0000 L CNN
+F 2 "SM0805" H 2600 3550 60  0001 C CNN
 	1    2600 3550
 	1    0    0    -1
@@
 F 0 "R61" V 2950 3300 50  0000 C CNN
 F 1 "10k" V 3050 3300 50  0000 C CNN
+F 2 "SM0805" H 2950 3300 60  0001 C CNN
 	1    2950 3300
 	0    1    1    0
@@
 F 0 "C37" H 2350 3650 50  0000 L CNN
 F 1 "0.01uF" H 2350 3450 50  0000 L CNN
+F 2 "SM0805" H 2300 3550 60  0001 C CNN
 	1    2300 3550
 	1    0    0    -1
@@
 F 0 "C49" H 7500 3600 50  0000 L CNN
 F 1 "10uF" H 7500 3400 50  0000 L CNN
+F 2 "SM0805" H 7450 3500 60  0001 C CNN
 	1    7450 3500
 	1    0    0    -1
@@
 F 0 "C48" H 7050 3600 50  0000 L CNN
 F 1 "150uF" H 7050 3400 50  0000 L CNN
+F 2 "CP10" H 7000 3500 60  0001 C CNN
 	1    7000 3500
 	1    0    0    -1
@@
 F 0 "R67" V 5850 2050 50  0000 C CNN
 F 1 "0.025" V 5950 2050 50  0000 C CNN
+F 2 "SM0805" H 5850 2050 60  0001 C CNN
 	1    5850 2050
 	1    0    0    -1
@@
 F 0 "U11" H 4950 2650 60  0000 C CNN
 F 1 "LTC1771" H 4600 3650 60  0000 C CNN
+F 2 "MSOP8" H 4600 3150 60  0001 C CNN
 	1    4600 3150
 	1    0    0    -1
