File: schematics/kicad_schematics/power_supply.sch (KiCad schematic (older format))
At the start: 28 parts, among them Q3 MOSFET_N, Q4 NMOS, U10 LTC3827, U11 LTC1771

Commit message: modified pinout on em406, update schematic, and modified pinout on S08 and SSOT6
Parts:
- C44: footprint SM0805 -> 10uf_Tantulum_Capacitor
- C45, C46: footprint SM1210L -> 100uf_Capacitor_Electrolytic
- C48: footprint CP10 -> 150uf_Capacitor_Electrolytic
- D15, D16: footprint SC-59 -> DO-124AB-DIODE
- Q4: footprint -SO-08 -> IRF8714PbF
Changed lines of the file:
@@
-EESchema Schematic File Version 2  date Sun 14 Mar 2010 03:28:34 PM EDT
+EESchema Schematic File Version 2  date Sun 14 Mar 2010 03:55:01 PM EDT
 LIBS:power
 LIBS:device
@@
 F 0 "C44" H 6000 5400 50  0000 L CNN
 F 1 "10uF" H 6000 5200 50  0000 L CNN
-F 2 "SM0805" H 5950 5300 60  0001 C CNN
+F 2 "10uf_Tantulum_Capacitor" H 5950 5300 60  0001 C CNN
 	1    5950 5300
 	1    0    0    -1
@@
 F 0 "C46" H 6650 6200 50  0000 L CNN
 F 1 "100uF" H 6650 6000 50  0000 L CNN
-F 2 "SM1210L" H 6600 6100 60  0001 C CNN
+F 2 "100uf_Capacitor_Electrolytic" H 6600 6100 60  0001 C CNN
 	1    6600 6100
 	1    0    0    -1
@@
 F 0 "C45" H 6300 6200 50  0000 L CNN
 F 1 "100uF" H 6300 6000 50  0000 L CNN
-F 2 "SM1210L" H 6250 6100 60  0001 C CNN
+F 2 "100uf_Capacitor_Electrolytic" H 6250 6100 60  0001 C CNN
 	1    6250 6100
 	1    0    0    -1
@@
 F 0 "D16" H 5950 5900 40  0000 C CNN
 F 1 "DIODESCH" H 5950 5700 40  0000 C CNN
-F 2 "SC-59" H 5950 5800 60  0001 C CNN
+F 2 "DO-124AB-DIODE" H 5950 5800 60  0001 C CNN
 	1    5950 5800
 	1    0    0    -1
@@
 F 0 "C48" H 7050 3600 50  0000 L CNN
 F 1 "150uF" H 7050 3400 50  0000 L CNN
-F 2 "CP10" H 7000 3500 60  0001 C CNN
+F 2 "150uf_Capacitor_Electrolytic" H 7000 3500 60  0001 C CNN
 	1    7000 3500
 	1    0    0    -1
@@
 F 0 "D15" H 5850 3550 40  0000 C CNN
 F 1 "DIODESCH" H 5850 3350 40  0000 C CNN
-F 2 "SC-59" H 5850 3450 60  0001 C CNN
+F 2 "DO-124AB-DIODE" H 5850 3450 60  0001 C CNN
 	1    5850 3450
 	0    -1   -1   0
@@
 F 0 "Q4" H 6000 2600 60  0000 R CNN
 F 1 "NMOS" H 6150 2700 60  0000 R CNN
-F 2 "-SO-08" H 5750 2700 60  0001 C CNN
+F 2 "IRF8714PbF" H 5750 2700 60  0001 C CNN
 	1    5750 2700
 	1    0    0    -1

Commit message: Modified power libraries. Now using custom power.lib. This is important Removed outdated crystal libaries Changed some caps to 0603 mounts started PCB layout
Parts:
- C37, C38, C39, C40, C41, C42, C43, C47, C49, R61, R62, R63, R64, R65, R66, R67: footprint SM0805 -> SM0805-CUSTOM
Changed lines of the file:
@@
-EESchema Schematic File Version 2  date Mon 15 Mar 2010 09:49:52 PM EDT
+EESchema Schematic File Version 2  date Tue 16 Mar 2010 05:07:11 PM EDT
 LIBS:power
 LIBS:device
@@
 F 0 "C40" H 2700 4900 50  0000 L CNN
 F 1 "47pF" H 2700 4700 50  0000 L CNN
-F 2 "SM0805" H 2650 4800 60  0001 C CNN
+F 2 "SM0805-CUSTOM" H 2650 4800 60  0001 C CNN
 	1    2650 4800
 	0    1    1    0
@@
 F 0 "C38" H 2450 5150 50  0000 L CNN
 F 1 "1.8nF" H 2450 4950 50  0000 L CNN
-F 2 "SM0805" H 2400 5050 60  0001 C CNN
+F 2 "SM0805-CUSTOM" H 2400 5050 60  0001 C CNN
 	1    2400 5050
 	0    1    1    0
@@
 F 0 "R62" V 3030 5050 50  0000 C CNN
 F 1 "17.4K" V 2950 5050 50  0000 C CNN
-F 2 "SM0805" H 2950 5050 60  0001 C CNN
+F 2 "SM0805-CUSTOM" H 2950 5050 60  0001 C CNN
 	1    2950 5050
 	0    1    1    0
@@
 F 0 "C41" H 3300 6250 50  0000 L CNN
 F 1 "5pF" H 3300 6050 50  0000 L CNN
-F 2 "SM0805" H 3250 6150 60  0001 C CNN
+F 2 "SM0805-CUSTOM" H 3250 6150 60  0001 C CNN
 	1    3250 6150
 	1    0    0    -1
@@
 F 0 "R63" V 3250 5650 50  0000 C CNN
 F 1 "11k 1%" V 3350 5650 50  0000 C CNN
-F 2 "SM0805" H 3250 5650 60  0001 C CNN
+F 2 "SM0805-CUSTOM" H 3250 5650 60  0001 C CNN
 	1    3250 5650
 	0    1    1    0
@@
 F 0 "R65" V 3550 6150 50  0000 C CNN
 F 1 "34.8k 1%" V 3650 6150 50  0000 C CNN
-F 2 "SM0805" H 3550 6150 60  0001 C CNN
+F 2 "SM0805-CUSTOM" H 3550 6150 60  0001 C CNN
 	1    3550 6150
 	1    0    0    -1
@@
 F 0 "C43" H 4350 6450 50  0000 L CNN
 F 1 "1nF" H 4350 6250 50  0000 L CNN
-F 2 "SM0805" H 4300 6350 60  0001 C CNN
+F 2 "SM0805-CUSTOM" H 4300 6350 60  0001 C CNN
 	1    4300 6350
 	1    0    0    -1
@@
 F 0 "C47" H 7000 6200 50  0000 L CNN
 F 1 "10uF" H 7000 6000 50  0000 L CNN
-F 2 "SM0805" H 6950 6100 60  0001 C CNN
+F 2 "SM0805-CUSTOM" H 6950 6100 60  0001 C CNN
 	1    6950 6100
 	1    0    0    -1
@@
 F 0 "C42" H 3450 3600 50  0000 L CNN
 F 1 "5pF" H 3450 3400 50  0000 L CNN
-F 2 "SM0805" H 3400 3500 60  0001 C CNN
+F 2 "SM0805-CUSTOM" H 3400 3500 60  0001 C CNN
 	1    3400 3500
 	0    1    1    0
@@
 F 0 "R66" V 4000 3750 50  0000 C CNN
 F 1 "1M 1%" V 4100 3750 50  0000 C CNN
-F 2 "SM0805" H 4000 3750 60  0001 C CNN
+F 2 "SM0805-CUSTOM" H 4000 3750 60  0001 C CNN
 	1    4000 3750
 	0    1    1    0
@@
 F 0 "R64" V 3400 3750 50  0000 C CNN
 F 1 "1.64M 1%" V 3500 3750 50  0000 C CNN
-F 2 "SM0805" H 3400 3750 60  0001 C CNN
+F 2 "SM0805-CUSTOM" H 3400 3750 60  0001 C CNN
 	1    3400 3750
 	0    1    1    0
@@
 F 0 "C39" H 2650 3650 50  0000 L CNN
 F 1 "220pF" H 2650 3450 50  0000 L CNN
-F 2 "SM0805" H 2600 3550 60  0001 C CNN
+F 2 "SM0805-CUSTOM" H 2600 3550 60  0001 C CNN
 	1    2600 3550
 	1    0    0    -1
@@
 F 0 "R61" V 2950 3300 50  0000 C CNN
 F 1 "10k" V 3050 3300 50  0000 C CNN
-F 2 "SM0805" H 2950 3300 60  0001 C CNN
+F 2 "SM0805-CUSTOM" H 2950 3300 60  0001 C CNN
 	1    2950 3300
 	0    1    1    0
@@
 F 0 "C37" H 2350 3650 50  0000 L CNN
 F 1 "0.01uF" H 2350 3450 50  0000 L CNN
-F 2 "SM0805" H 2300 3550 60  0001 C CNN
+F 2 "SM0805-CUSTOM" H 2300 3550 60  0001 C CNN
 	1    2300 3550
 	1    0    0    -1
@@
 F 0 "C49" H 7500 3600 50  0000 L CNN
 F 1 "10uF" H 7500 3400 50  0000 L CNN
-F 2 "SM0805" H 7450 3500 60  0001 C CNN
+F 2 "SM0805-CUSTOM" H 7450 3500 60  0001 C CNN
 	1    7450 3500
 	1    0    0    -1
@@
 F 0 "R67" V 5850 2050 50  0000 C CNN
 F 1 "0.025" V 5950 2050 50  0000 C CNN
-F 2 "SM0805" H 5850 2050 60  0001 C CNN
+F 2 "SM0805-CUSTOM" H 5850 2050 60  0001 C CNN
 	1    5850 2050
 	1    0    0    -1

Commit message: modified SM0603 and schematics, along with lots of work done on PCB layout design
Parts:
- C45, C46: value 100uF -> 150uF
Changed lines of the file:
@@
-EESchema Schematic File Version 2  date Tue 16 Mar 2010 05:07:11 PM EDT
+EESchema Schematic File Version 2  date Tue 16 Mar 2010 10:34:52 PM EDT
 LIBS:power
 LIBS:device
@@
 Sheet 3 5
 Title ""
-Date "16 mar 2010"
+Date "17 mar 2010"
 Rev ""
 Comp ""
@@
 P 6600 6100
 F 0 "C46" H 6650 6200 50  0000 L CNN
-F 1 "100uF" H 6650 6000 50  0000 L CNN
+F 1 "150uF" H 6650 6000 50  0000 L CNN
 F 2 "100uf_Capacitor_Electrolytic" H 6600 6100 60  0001 C CNN
 	1    6600 6100
@@
 P 6250 6100
 F 0 "C45" H 6300 6200 50  0000 L CNN
-F 1 "100uF" H 6300 6000 50  0000 L CNN
+F 1 "150uF" H 6300 6000 50  0000 L CNN
 F 2 "100uf_Capacitor_Electrolytic" H 6250 6100 60  0001 C CNN
 	1    6250 6100

Commit message: made some major changes to the PCB layout
Parts:
- C45, C46: footprint 100uf_Capacitor_Electrolytic -> 150uf_Capacitor_Electrolytic
Changed lines of the file:
@@
-EESchema Schematic File Version 2  date Tue 16 Mar 2010 10:34:52 PM EDT
+EESchema Schematic File Version 2  date Wed 17 Mar 2010 01:46:08 PM EDT
 LIBS:power
 LIBS:device
@@
 F 0 "C46" H 6650 6200 50  0000 L CNN
 F 1 "150uF" H 6650 6000 50  0000 L CNN
-F 2 "100uf_Capacitor_Electrolytic" H 6600 6100 60  0001 C CNN
+F 2 "150uf_Capacitor_Electrolytic" H 6600 6100 60  0001 C CNN
 	1    6600 6100
 	1    0    0    -1
@@
 F 0 "C45" H 6300 6200 50  0000 L CNN
 F 1 "150uF" H 6300 6000 50  0000 L CNN
-F 2 "100uf_Capacitor_Electrolytic" H 6250 6100 60  0001 C CNN
+F 2 "150uf_Capacitor_Electrolytic" H 6250 6100 60  0001 C CNN
 	1    6250 6100
 	1    0    0    -1
