File: schematics/kicad_schematics/wiznet_network.sch (KiCad schematic (older format))
At the start: 49 parts, among them SW4 DIPS_03, U6 W5300, U7 RD1-125BAG1A, X4 25MHz

Commit message: Fixed some data modules
Parts:
- D19: renamed from D?; footprint (none) -> SC-59
Changed lines of the file:
@@
-EESchema Schematic File Version 2  date Sat 13 Mar 2010 02:28:46 PM EST
+EESchema Schematic File Version 2  date Sat 13 Mar 2010 03:45:55 PM EST
 LIBS:power
 LIBS:device
@@
 	3800 7900 3800 7700
 $Comp
-L 1SS181 D?
+L 1SS181 D19
 U 1 1 4B9BE6A8
 P 10550 1950
-F 0 "D?" H 10550 2350 40  0000 C CNN
+F 0 "D19" H 10550 2350 40  0000 C CNN
 F 1 "1SS181" H 10550 1850 40  0000 C CNN
+F 2 "SC-59" H 10550 1950 60  0001 C CNN
 	1    10550 1950
 	1    0    0    -1
@@
 NoConn ~ 2250 6700
 $Comp
-L GND #PWR49
+L GND #PWR037
 U 1 1 4B984217
 P 10950 7350
-F 0 "#PWR49" H 10950 7350 30  0001 C CNN
+F 0 "#PWR037" H 10950 7350 30  0001 C CNN
 F 1 "GND" H 10950 7280 30  0001 C CNN
 	1    10950 7350
@@
 A0 - GND IN 16-BIT MODE
 $Comp
-L GND #PWR33
+L GND #PWR038
 U 1 1 4B903065
 P 1400 5250
-F 0 "#PWR33" H 1400 5250 30  0001 C CNN
+F 0 "#PWR038" H 1400 5250 30  0001 C CNN
 F 1 "GND" H 1400 5180 30  0001 C CNN
 	1    1400 5250
@@
 $EndComp
 $Comp
-L GND #PWR42
+L GND #PWR039
 U 1 1 4B6DC2F1
 P 8350 9700
-F 0 "#PWR42" H 8350 9700 30  0001 C CNN
+F 0 "#PWR039" H 8350 9700 30  0001 C CNN
 F 1 "GND" H 8350 9630 30  0001 C CNN
 	1    8350 9700
@@
 $EndComp
 $Comp
-L GNDA #PWR43
+L GNDA #PWR040
 U 1 1 4B6DC0F8
 P 9450 4750
-F 0 "#PWR43" H 9450 4750 40  0001 C CNN
+F 0 "#PWR040" H 9450 4750 40  0001 C CNN
 F 1 "GNDA" H 9450 4680 40  0000 C CNN
 	1    9450 4750
@@
 $EndComp
 $Comp
-L GNDA #PWR46
+L GNDA #PWR041
 U 1 1 4B6DC0D3
 P 10150 7350
-F 0 "#PWR46" H 10150 7350 40  0001 C CNN
+F 0 "#PWR041" H 10150 7350 40  0001 C CNN
 F 1 "GNDA" H 10150 7280 40  0000 C CNN
 	1    10150 7350
@@
 $EndComp
 $Comp
-L GNDA #PWR44
+L GNDA #PWR042
 U 1 1 4B6DC05D
 P 9450 7450
-F 0 "#PWR44" H 9450 7450 40  0001 C CNN
+F 0 "#PWR042" H 9450 7450 40  0001 C CNN
 F 1 "GNDA" H 9450 7380 40  0000 C CNN
 	1    9450 7450
@@
 $EndComp
 $Comp
-L GND #PWR58
+L GND #PWR043
 U 1 1 4B6DB951
 P 13150 5650
-F 0 "#PWR58" H 13150 5650 30  0001 C CNN
+F 0 "#PWR043" H 13150 5650 30  0001 C CNN
 F 1 "GND" H 13150 5580 30  0001 C CNN
 	1    13150 5650
@@
 $EndComp
 $Comp
-L GNDA #PWR63
+L GNDA #PWR044
 U 1 1 4B6DB94B
 P 14400 5650
-F 0 "#PWR63" H 14400 5650 40  0001 C CNN
+F 0 "#PWR044" H 14400 5650 40  0001 C CNN
 F 1 "GNDA" H 14400 5580 40  0000 C CNN
 	1    14400 5650
@@
 1V8_OUT
 $Comp
-L GNDA #PWR61
+L GNDA #PWR045
 U 1 1 4B6DB901
 P 14400 4200
-F 0 "#PWR61" H 14400 4200 40  0001 C CNN
+F 0 "#PWR045" H 14400 4200 40  0001 C CNN
 F 1 "GNDA" H 14400 4130 40  0000 C CNN
 	1    14400 4200
@@
 $EndComp
 $Comp
-L GND #PWR56
+L GND #PWR046
 U 1 1 4B6DB886
 P 13150 4200
-F 0 "#PWR56" H 13150 4200 30  0001 C CNN
+F 0 "#PWR046" H 13150 4200 30  0001 C CNN
 F 1 "GND" H 13150 4130 30  0001 C CNN
 	1    13150 4200
@@
 $EndComp
 $Comp
-L GNDA #PWR66
+L GNDA #PWR047
 U 1 1 4B6DB84F
 P 15850 1750
-F 0 "#PWR66" H 15850 1750 40  0001 C CNN
+F 0 "#PWR047" H 15850 1750 40  0001 C CNN
 F 1 "GNDA" H 15850 1680 40  0000 C CNN
 	1    15850 1750
@@
 $EndComp
 $Comp
-L GND #PWR65
+L GND #PWR048
 U 1 1 4B6DB842
 P 15250 1750
-F 0 "#PWR65" H 15250 1750 30  0001 C CNN
+F 0 "#PWR048" H 15250 1750 30  0001 C CNN
 F 1 "GND" H 15250 1680 30  0001 C CNN
 	1    15250 1750
@@
 $EndComp
 $Comp
-L GND #PWR54
+L GND #PWR049
 U 1 1 4B6DB7C7
 P 13150 3150
-F 0 "#PWR54" H 13150 3150 30  0001 C CNN
+F 0 "#PWR049" H 13150 3150 30  0001 C CNN
 F 1 "GND" H 13150 3080 30  0001 C CNN
 	1    13150 3150
@@
 $EndComp
 $Comp
-L GND #PWR52
+L GND #PWR050
 U 1 1 4B6DB77B
 P 13150 2100
-F 0 "#PWR52" H 13150 2100 30  0001 C CNN
+F 0 "#PWR050" H 13150 2100 30  0001 C CNN
 F 1 "GND" H 13150 2030 30  0001 C CNN
 	1    13150 2100
@@
 TEST_MODE3
 $Comp
-L GND #PWR34
+L GND #PWR051
 U 1 1 4B6DB150
 P 2050 7550
-F 0 "#PWR34" H 2050 7550 30  0001 C CNN
+F 0 "#PWR051" H 2050 7550 30  0001 C CNN
 F 1 "GND" H 2050 7480 30  0001 C CNN
 	1    2050 7550
@@
 $EndComp
 $Comp
-L GND #PWR40
+L GND #PWR052
 U 1 1 4B6DAEFD
 P 5200 7900
-F 0 "#PWR40" H 5200 7900 30  0001 C CNN
+F 0 "#PWR052" H 5200 7900 30  0001 C CNN
 F 1 "GND" H 5200 7830 30  0001 C CNN
 	1    5200 7900
@@
 $EndComp
 $Comp
-L GND #PWR41
+L GND #PWR053
 U 1 1 4B6DAEC0
 P 7100 2400
-F 0 "#PWR41" H 7100 2400 30  0001 C CNN
+F 0 "#PWR053" H 7100 2400 30  0001 C CNN
 F 1 "GND" H 7100 2330 30  0001 C CNN
 	1    7100 2400
@@
 $EndComp
 $Comp
-L GNDA #PWR37
+L GNDA #PWR054
 U 1 1 4B6DAEA9
 P 3800 7900
-F 0 "#PWR37" H 3800 7900 40  0001 C CNN
+F 0 "#PWR054" H 3800 7900 40  0001 C CNN
 F 1 "GNDA" H 3800 7830 40  0000 C CNN
 	1    3800 7900

Commit message: added npn datasheet
Parts:
- L2, L3, L4: footprint (none) -> SM0805
Changed lines of the file:
@@
-EESchema Schematic File Version 2  date Sat 13 Mar 2010 03:45:55 PM EST
+EESchema Schematic File Version 2  date Sat 13 Mar 2010 04:13:45 PM EST
 LIBS:power
 LIBS:device
@@
 F 0 "L3" V 13850 5100 40  0000 C CNN
 F 1 "1uH" V 14000 5100 40  0000 C CNN
+F 2 "SM0805" H 13900 5100 60  0001 C CNN
 	1    13900 5100
 	0    -1   -1   0
@@
 F 0 "L2" V 13850 3650 40  0000 C CNN
 F 1 "1uH" V 14000 3650 40  0000 C CNN
+F 2 "SM0805" H 13900 3650 60  0001 C CNN
 	1    13900 3650
 	0    -1   -1   0
@@
 F 0 "L4" V 15500 1650 40  0000 C CNN
 F 1 "1uH" V 15650 1650 40  0000 C CNN
+F 2 "SM0805" H 15550 1650 60  0001 C CNN
 	1    15550 1650
 	0    -1   -1   0

Commit message: added datasheets and modified schematic components for new dip switches
Parts:
- SW4: PART (none) -> 219-02-3MSTR
Changed lines of the file:
@@
-EESchema Schematic File Version 2  date Sat 13 Mar 2010 04:13:45 PM EST
+EESchema Schematic File Version 2  date Sun 14 Mar 2010 12:34:26 PM EDT
 LIBS:power
 LIBS:device
@@
 Sheet 4 5
 Title ""
-Date "13 mar 2010"
+Date "14 mar 2010"
 Rev ""
 Comp ""
@@
 NoConn ~ 2250 6700
 $Comp
-L GND #PWR037
+L GND #PWR036
 U 1 1 4B984217
 P 10950 7350
-F 0 "#PWR037" H 10950 7350 30  0001 C CNN
+F 0 "#PWR036" H 10950 7350 30  0001 C CNN
 F 1 "GND" H 10950 7280 30  0001 C CNN
 	1    10950 7350
@@
 A0 - GND IN 16-BIT MODE
 $Comp
-L GND #PWR038
+L GND #PWR037
 U 1 1 4B903065
 P 1400 5250
-F 0 "#PWR038" H 1400 5250 30  0001 C CNN
+F 0 "#PWR037" H 1400 5250 30  0001 C CNN
 F 1 "GND" H 1400 5180 30  0001 C CNN
 	1    1400 5250
@@
 $EndComp
 $Comp
-L GND #PWR039
+L GND #PWR038
 U 1 1 4B6DC2F1
 P 8350 9700
-F 0 "#PWR039" H 8350 9700 30  0001 C CNN
+F 0 "#PWR038" H 8350 9700 30  0001 C CNN
 F 1 "GND" H 8350 9630 30  0001 C CNN
 	1    8350 9700
@@
 $EndComp
 $Comp
-L GNDA #PWR040
+L GNDA #PWR039
 U 1 1 4B6DC0F8
 P 9450 4750
-F 0 "#PWR040" H 9450 4750 40  0001 C CNN
+F 0 "#PWR039" H 9450 4750 40  0001 C CNN
 F 1 "GNDA" H 9450 4680 40  0000 C CNN
 	1    9450 4750
@@
 $EndComp
 $Comp
-L GNDA #PWR041
+L GNDA #PWR040
 U 1 1 4B6DC0D3
 P 10150 7350
-F 0 "#PWR041" H 10150 7350 40  0001 C CNN
+F 0 "#PWR040" H 10150 7350 40  0001 C CNN
 F 1 "GNDA" H 10150 7280 40  0000 C CNN
 	1    10150 7350
@@
 $EndComp
 $Comp
-L -8V #PWR45
+L -8V #PWR43
 U 1 1 4B6DC0CC
 P 10150 4750
-F 0 "#PWR45" H 10150 4880 20  0001 C CNN
+F 0 "#PWR43" H 10150 4880 20  0001 C CNN
 F 1 "3V3A" H 10150 4850 30  0000 C CNN
 	1    10150 4750
@@
 $EndComp
 $Comp
-L GNDA #PWR042
+L GNDA #PWR041
 U 1 1 4B6DC05D
 P 9450 7450
-F 0 "#PWR042" H 9450 7450 40  0001 C CNN
+F 0 "#PWR041" H 9450 7450 40  0001 C CNN
 F 1 "GNDA" H 9450 7380 40  0000 C CNN
 	1    9450 7450
@@
 $EndComp
 $Comp
-L -8V #PWR47
+L -8V #PWR45
 U 1 1 4B6DC045
 P 10550 4750
-F 0 "#PWR47" H 10550 4880 20  0001 C CNN
+F 0 "#PWR45" H 10550 4880 20  0001 C CNN
 F 1 "3V3A" H 10550 4850 30  0000 C CNN
 	1    10550 4750
@@
 $EndComp
 $Comp
-L -8V #PWR64
+L -8V #PWR62
 U 1 1 4B6DBDDB
 P 14550 7150
-F 0 "#PWR64" H 14550 7280 20  0001 C CNN
+F 0 "#PWR62" H 14550 7280 20  0001 C CNN
 F 1 "3.3V" H 14550 7250 30  0000 C CNN
 	1    14550 7150
@@
 F 0 "SW4" V 14000 7350 60  0000 C CNN
 F 1 "DIPS_03" V 14400 7350 60  0000 C CNN
+F 4 "219-02-3MSTR" H 14200 7350 60  0001 C CNN "PART"
 	1    14200 7350
 	0    1    1    0
@@
 BIT16EN
 $Comp
-L -8V #PWR59
+L -8V #PWR57
 U 1 1 4B6DBBEE
 P 13400 8050
-F 0 "#PWR59" H 13400 8180 20  0001 C CNN
+F 0 "#PWR57" H 13400 8180 20  0001 C CNN
 F 1 "3.3V" H 13400 8150 30  0000 C CNN
 	1    13400 8050
@@
 $EndComp
 $Comp
-L -8V #PWR50
+L -8V #PWR48
 U 1 1 4B6DBBAB
 P 11450 2750
-F 0 "#PWR50" H 11450 2880 20  0001 C CNN
+F 0 "#PWR48" H 11450 2880 20  0001 C CNN
 F 1 "3.3V" H 11450 2850 30  0000 C CNN
 	1    11450 2750
@@
 /ACTLED
 $Comp
-L -8V #PWR48
+L -8V #PWR46
 U 1 1 4B6DBA93
 P 10950 1200
-F 0 "#PWR48" H 10950 1330 20  0001 C CNN
+F 0 "#PWR46" H 10950 1330 20  0001 C CNN
 F 1 "3.3V" H 10950 1300 30  0000 C CNN
 	1    10950 1200
@@
 $EndComp
 $Comp
-L GND #PWR043
+L GND #PWR042
 U 1 1 4B6DB951
 P 13150 5650
-F 0 "#PWR043" H 13150 5650 30  0001 C CNN
+F 0 "#PWR042" H 13150 5650 30  0001 C CNN
 F 1 "GND" H 13150 5580 30  0001 C CNN
 	1    13150 5650
@@
 $EndComp
 $Comp
-L -8V #PWR57
+L -8V #PWR55
 U 1 1 4B6DB950
 P 13150 4950
-F 0 "#PWR57" H 13150 5080 20  0001 C CNN
+F 0 "#PWR55" H 13150 5080 20  0001 C CNN
 F 1 "3.3V" H 13150 5050 30  0000 C CNN
 	1    13150 4950
@@
 $EndComp
 $Comp
-L -8V #PWR62
+L -8V #PWR60
 U 1 1 4B6DB94E
 P 14400 4950
-F 0 "#PWR62" H 14400 5080 20  0001 C CNN
+F 0 "#PWR60" H 14400 5080 20  0001 C CNN
 F 1 "3V3A" H 14400 5050 30  0000 C CNN
 	1    14400 4950
@@
 $EndComp
 $Comp
-L GNDA #PWR044
+L GNDA #PWR043
 U 1 1 4B6DB94B
 P 14400 5650
-F 0 "#PWR044" H 14400 5650 40  0001 C CNN
+F 0 "#PWR043" H 14400 5650 40  0001 C CNN
 F 1 "GNDA" H 14400 5580 40  0000 C CNN
 	1    14400 5650
@@
 1V8_OUT
 $Comp
-L GNDA #PWR045
+L GNDA #PWR044
 U 1 1 4B6DB901
 P 14400 4200
-F 0 "#PWR045" H 14400 4200 40  0001 C CNN
+F 0 "#PWR044" H 14400 4200 40  0001 C CNN
 F 1 "GNDA" H 14400 4130 40  0000 C CNN
 	1    14400 4200
@@
 $EndComp
 $Comp
-L -8V #PWR60
+L -8V #PWR58
 U 1 1 4B6DB8BA
 P 14400 3500
-F 0 "#PWR60" H 14400 3630 20  0001 C CNN
+F 0 "#PWR58" H 14400 3630 20  0001 C CNN
 F 1 "1V8A" H 14400 3600 30  0000 C CNN
 	1    14400 3500
@@
 $EndComp
 $Comp
-L -8V #PWR55
+L -8V #PWR53
 U 1 1 4B6DB887
 P 13150 3500
-F 0 "#PWR55" H 13150 3630 20  0001 C CNN
+F 0 "#PWR53" H 13150 3630 20  0001 C CNN
 F 1 "1V8D" H 13150 3600 30  0000 C CNN
 	1    13150 3500
@@
 $EndComp
 $Comp
-L GND #PWR046
+L GND #PWR045
 U 1 1 4B6DB886
 P 13150 4200
-F 0 "#PWR046" H 13150 4200 30  0001 C CNN
+F 0 "#PWR045" H 13150 4200 30  0001 C CNN
 F 1 "GND" H 13150 4130 30  0001 C CNN
 	1    13150 4200
@@
 $EndComp
 $Comp
-L GNDA #PWR047
+L GNDA #PWR046
 U 1 1 4B6DB84F
 P 15850 1750
-F 0 "#PWR047" H 15850 1750 40  0001 C CNN
+F 0 "#PWR046" H 15850 1750 40  0001 C CNN
 F 1 "GNDA" H 15850 1680 40  0000 C CNN
 	1    15850 1750
@@
 $EndComp
 $Comp
-L GND #PWR048
+L GND #PWR047
 U 1 1 4B6DB842
 P 15250 1750
-F 0 "#PWR048" H 15250 1750 30  0001 C CNN
+F 0 "#PWR047" H 15250 1750 30  0001 C CNN
 F 1 "GND" H 15250 1680 30  0001 C CNN
 	1    15250 1750
@@
 $EndComp
 $Comp
-L GND #PWR049
+L GND #PWR048
 U 1 1 4B6DB7C7
 P 13150 3150
-F 0 "#PWR049" H 13150 3150 30  0001 C CNN
+F 0 "#PWR048" H 13150 3150 30  0001 C CNN
 F 1 "GND" H 13150 3080 30  0001 C CNN
 	1    13150 3150
@@
 $EndComp
 $Comp
-L -8V #PWR53
+L -8V #PWR51
 U 1 1 4B6DB7C6
 P 13150 2450
-F 0 "#PWR53" H 13150 2580 20  0001 C CNN
+F 0 "#PWR51" H 13150 2580 20  0001 C CNN
 F 1 "1V8D" H 13150 2550 30  0000 C CNN
 	1    13150 2450
@@
 $EndComp
 $Comp
-L -8V #PWR51
+L -8V #PWR49
 U 1 1 4B6DB78D
 P 13150 1400
-F 0 "#PWR51" H 13150 1530 20  0001 C CNN
+F 0 "#PWR49" H 13150 1530 20  0001 C CNN
 F 1 "3.3V" H 13150 1500 30  0000 C CNN
 	1    13150 1400
@@
 $EndComp
 $Comp
-L GND #PWR050
+L GND #PWR049
 U 1 1 4B6DB77B
 P 13150 2100
-F 0 "#PWR050" H 13150 2100 30  0001 C CNN
+F 0 "#PWR049" H 13150 2100 30  0001 C CNN
 F 1 "GND" H 13150 2030 30  0001 C CNN
 	1    13150 2100
@@
 TEST_MODE3
 $Comp
-L GND #PWR051
+L GND #PWR050
 U 1 1 4B6DB150
 P 2050 7550
-F 0 "#PWR051" H 2050 7550 30  0001 C CNN
+F 0 "#PWR050" H 2050 7550 30  0001 C CNN
 F 1 "GND" H 2050 7480 30  0001 C CNN
 	1    2050 7550
@@
 VCC3A3
 $Comp
-L -8V #PWR39
+L -8V #PWR37
 U 1 1 4B6DB004
 P 4650 1250
-F 0 "#PWR39" H 4650 1380 20  0001 C CNN
+F 0 "#PWR37" H 4650 1380 20  0001 C CNN
 F 1 "1V8D" H 4650 1350 30  0000 C CNN
 	1    4650 1250
@@
 $EndComp
 $Comp
-L -8V #PWR38
+L -8V #PWR36
 U 1 1 4B6DAFF8
 P 4050 1250
-F 0 "#PWR38" H 4050 1380 20  0001 C CNN
+F 0 "#PWR36" H 4050 1380 20  0001 C CNN
 F 1 "3.3V" H 4050 1350 30  0000 C CNN
 	1    4050 1250
@@
 $EndComp
 $Comp
-L -8V #PWR36
+L -8V #PWR34
 U 1 1 4B6DAFF2
 P 3750 1250
-F 0 "#PWR36" H 3750 1380 20  0001 C CNN
+F 0 "#PWR34" H 3750 1380 20  0001 C CNN
 F 1 "1V8A" H 3750 1350 30  0000 C CNN
 	1    3750 1250
@@
 $EndComp
 $Comp
-L -8V #PWR35
+L -8V #PWR33
 U 1 1 4B6DAFC6
 P 3550 1250
-F 0 "#PWR35" H 3550 1380 20  0001 C CNN
+F 0 "#PWR33" H 3550 1380 20  0001 C CNN
 F 1 "3V3A" H 3550 1350 30  0000 C CNN
 	1    3550 1250
@@
 $EndComp
 $Comp
-L GND #PWR052
+L GND #PWR051
 U 1 1 4B6DAEFD
 P 5200 7900
-F 0 "#PWR052" H 5200 7900 30  0001 C CNN
+F 0 "#PWR051" H 5200 7900 30  0001 C CNN
 F 1 "GND" H 5200 7830 30  0001 C CNN
 	1    5200 7900
@@
 $EndComp
 $Comp
-L GND #PWR053
+L GND #PWR052
 U 1 1 4B6DAEC0
 P 7100 2400
-F 0 "#PWR053" H 7100 2400 30  0001 C CNN
+F 0 "#PWR052" H 7100 2400 30  0001 C CNN
 F 1 "GND" H 7100 2330 30  0001 C CNN
 	1    7100 2400
@@
 $EndComp
 $Comp
-L GNDA #PWR054
+L GNDA #PWR053
 U 1 1 4B6DAEA9
 P 3800 7900
-F 0 "#PWR054" H 3800 7900 40  0001 C CNN
+F 0 "#PWR053" H 3800 7900 40  0001 C CNN
 F 1 "GNDA" H 3800 7830 40  0000 C CNN
 	1    3800 7900

Commit message: Updated schematics removing spaces
Parts:
- SW4: footprint (none) -> SPST-DIP-219-3MSTR
- X4: footprint (none) -> 25Mhz-Crystal
Changed lines of the file:
@@
-EESchema Schematic File Version 2  date Sun 14 Mar 2010 12:34:26 PM EDT
+EESchema Schematic File Version 2  date Sun 14 Mar 2010 01:29:31 PM EDT
 LIBS:power
 LIBS:device
@@
 NoConn ~ 2250 6700
 $Comp
-L GND #PWR036
+L GND #PWR038
 U 1 1 4B984217
 P 10950 7350
-F 0 "#PWR036" H 10950 7350 30  0001 C CNN
+F 0 "#PWR038" H 10950 7350 30  0001 C CNN
 F 1 "GND" H 10950 7280 30  0001 C CNN
 	1    10950 7350
@@
 A0 - GND IN 16-BIT MODE
 $Comp
-L GND #PWR037
+L GND #PWR039
 U 1 1 4B903065
 P 1400 5250
-F 0 "#PWR037" H 1400 5250 30  0001 C CNN
+F 0 "#PWR039" H 1400 5250 30  0001 C CNN
 F 1 "GND" H 1400 5180 30  0001 C CNN
 	1    1400 5250
@@
 $EndComp
 $Comp
-L GND #PWR038
+L GND #PWR040
 U 1 1 4B6DC2F1
 P 8350 9700
-F 0 "#PWR038" H 8350 9700 30  0001 C CNN
+F 0 "#PWR040" H 8350 9700 30  0001 C CNN
 F 1 "GND" H 8350 9630 30  0001 C CNN
 	1    8350 9700
@@
 F 0 "X4" V 9300 9300 60  0000 C CNN
 F 1 "25MHz" V 8950 9350 60  0000 C CNN
+F 2 "25Mhz-Crystal" H 9150 9200 60  0001 C CNN
 	1    9150 9200
 	0    -1   -1   0
@@
 $EndComp
 $Comp
-L GNDA #PWR039
+L GNDA #PWR041
 U 1 1 4B6DC0F8
 P 9450 4750
-F 0 "#PWR039" H 9450 4750 40  0001 C CNN
+F 0 "#PWR041" H 9450 4750 40  0001 C CNN
 F 1 "GNDA" H 9450 4680 40  0000 C CNN
 	1    9450 4750
@@
 $EndComp
 $Comp
-L GNDA #PWR040
+L GNDA #PWR042
 U 1 1 4B6DC0D3
 P 10150 7350
-F 0 "#PWR040" H 10150 7350 40  0001 C CNN
+F 0 "#PWR042" H 10150 7350 40  0001 C CNN
 F 1 "GNDA" H 10150 7280 40  0000 C CNN
 	1    10150 7350
@@
 $EndComp
 $Comp
-L -8V #PWR43
+L -8V #PWR45
 U 1 1 4B6DC0CC
 P 10150 4750
-F 0 "#PWR43" H 10150 4880 20  0001 C CNN
+F 0 "#PWR45" H 10150 4880 20  0001 C CNN
 F 1 "3V3A" H 10150 4850 30  0000 C CNN
 	1    10150 4750
@@
 $EndComp
 $Comp
-L GNDA #PWR041
+L GNDA #PWR043
 U 1 1 4B6DC05D
 P 9450 7450
-F 0 "#PWR041" H 9450 7450 40  0001 C CNN
+F 0 "#PWR043" H 9450 7450 40  0001 C CNN
 F 1 "GNDA" H 9450 7380 40  0000 C CNN
 	1    9450 7450
@@
 $EndComp
 $Comp
-L -8V #PWR45
+L -8V #PWR47
 U 1 1 4B6DC045
 P 10550 4750
-F 0 "#PWR45" H 10550 4880 20  0001 C CNN
+F 0 "#PWR47" H 10550 4880 20  0001 C CNN
 F 1 "3V3A" H 10550 4850 30  0000 C CNN
 	1    10550 4750
@@
 $EndComp
 $Comp
-L -8V #PWR62
+L -8V #PWR64
 U 1 1 4B6DBDDB
 P 14550 7150
-F 0 "#PWR62" H 14550 7280 20  0001 C CNN
+F 0 "#PWR64" H 14550 7280 20  0001 C CNN
 F 1 "3.3V" H 14550 7250 30  0000 C CNN
 	1    14550 7150
@@
 F 0 "SW4" V 14000 7350 60  0000 C CNN
 F 1 "DIPS_03" V 14400 7350 60  0000 C CNN
+F 2 "SPST-DIP-219-3MSTR" H 14200 7350 60  0001 C CNN
 F 4 "219-02-3MSTR" H 14200 7350 60  0001 C CNN "PART"
 	1    14200 7350
@@
 BIT16EN
 $Comp
-L -8V #PWR57
+L -8V #PWR59
 U 1 1 4B6DBBEE
 P 13400 8050
-F 0 "#PWR57" H 13400 8180 20  0001 C CNN
+F 0 "#PWR59" H 13400 8180 20  0001 C CNN
 F 1 "3.3V" H 13400 8150 30  0000 C CNN
 	1    13400 8050
@@
 $EndComp
 $Comp
-L -8V #PWR48
+L -8V #PWR50
 U 1 1 4B6DBBAB
 P 11450 2750
-F 0 "#PWR48" H 11450 2880 20  0001 C CNN
+F 0 "#PWR50" H 11450 2880 20  0001 C CNN
 F 1 "3.3V" H 11450 2850 30  0000 C CNN
 	1    11450 2750
@@
 /ACTLED
 $Comp
-L -8V #PWR46
+L -8V #PWR48
 U 1 1 4B6DBA93
 P 10950 1200
-F 0 "#PWR46" H 10950 1330 20  0001 C CNN
+F 0 "#PWR48" H 10950 1330 20  0001 C CNN
 F 1 "3.3V" H 10950 1300 30  0000 C CNN
 	1    10950 1200
@@
 $EndComp
 $Comp
-L GND #PWR042
+L GND #PWR044
 U 1 1 4B6DB951
 P 13150 5650
-F 0 "#PWR042" H 13150 5650 30  0001 C CNN
+F 0 "#PWR044" H 13150 5650 30  0001 C CNN
 F 1 "GND" H 13150 5580 30  0001 C CNN
 	1    13150 5650
@@
 $EndComp
 $Comp
-L -8V #PWR55
+L -8V #PWR57
 U 1 1 4B6DB950
 P 13150 4950
-F 0 "#PWR55" H 13150 5080 20  0001 C CNN
+F 0 "#PWR57" H 13150 5080 20  0001 C CNN
 F 1 "3.3V" H 13150 5050 30  0000 C CNN
 	1    13150 4950
@@
 $EndComp
 $Comp
-L -8V #PWR60
+L -8V #PWR62
 U 1 1 4B6DB94E
 P 14400 4950
-F 0 "#PWR60" H 14400 5080 20  0001 C CNN
+F 0 "#PWR62" H 14400 5080 20  0001 C CNN
 F 1 "3V3A" H 14400 5050 30  0000 C CNN
 	1    14400 4950
@@
 $EndComp
 $Comp
-L GNDA #PWR043
+L GNDA #PWR045
 U 1 1 4B6DB94B
 P 14400 5650
-F 0 "#PWR043" H 14400 5650 40  0001 C CNN
+F 0 "#PWR045" H 14400 5650 40  0001 C CNN
 F 1 "GNDA" H 14400 5580 40  0000 C CNN
 	1    14400 5650
@@
 1V8_OUT
 $Comp
-L GNDA #PWR044
+L GNDA #PWR046
 U 1 1 4B6DB901
 P 14400 4200
-F 0 "#PWR044" H 14400 4200 40  0001 C CNN
+F 0 "#PWR046" H 14400 4200 40  0001 C CNN
 F 1 "GNDA" H 14400 4130 40  0000 C CNN
 	1    14400 4200
@@
 $EndComp
 $Comp
-L -8V #PWR58
+L -8V #PWR60
 U 1 1 4B6DB8BA
 P 14400 3500
-F 0 "#PWR58" H 14400 3630 20  0001 C CNN
+F 0 "#PWR60" H 14400 3630 20  0001 C CNN
 F 1 "1V8A" H 14400 3600 30  0000 C CNN
 	1    14400 3500
@@
 $EndComp
 $Comp
-L -8V #PWR53
+L -8V #PWR55
 U 1 1 4B6DB887
 P 13150 3500
-F 0 "#PWR53" H 13150 3630 20  0001 C CNN
+F 0 "#PWR55" H 13150 3630 20  0001 C CNN
 F 1 "1V8D" H 13150 3600 30  0000 C CNN
 	1    13150 3500
@@
 $EndComp
 $Comp
-L GND #PWR045
+L GND #PWR047
 U 1 1 4B6DB886
 P 13150 4200
-F 0 "#PWR045" H 13150 4200 30  0001 C CNN
+F 0 "#PWR047" H 13150 4200 30  0001 C CNN
 F 1 "GND" H 13150 4130 30  0001 C CNN
 	1    13150 4200
@@
 $EndComp
 $Comp
-L GNDA #PWR046
+L GNDA #PWR048
 U 1 1 4B6DB84F
 P 15850 1750
-F 0 "#PWR046" H 15850 1750 40  0001 C CNN
+F 0 "#PWR048" H 15850 1750 40  0001 C CNN
 F 1 "GNDA" H 15850 1680 40  0000 C CNN
 	1    15850 1750
@@
 $EndComp
 $Comp
-L GND #PWR047
+L GND #PWR049
 U 1 1 4B6DB842
 P 15250 1750
-F 0 "#PWR047" H 15250 1750 30  0001 C CNN
+F 0 "#PWR049" H 15250 1750 30  0001 C CNN
 F 1 "GND" H 15250 1680 30  0001 C CNN
 	1    15250 1750
@@
 $EndComp
 $Comp
-L GND #PWR048
+L GND #PWR050
 U 1 1 4B6DB7C7
 P 13150 3150
-F 0 "#PWR048" H 13150 3150 30  0001 C CNN
+F 0 "#PWR050" H 13150 3150 30  0001 C CNN
 F 1 "GND" H 13150 3080 30  0001 C CNN
 	1    13150 3150
@@
 $EndComp
 $Comp
-L -8V #PWR51
+L -8V #PWR53
 U 1 1 4B6DB7C6
 P 13150 2450
-F 0 "#PWR51" H 13150 2580 20  0001 C CNN
+F 0 "#PWR53" H 13150 2580 20  0001 C CNN
 F 1 "1V8D" H 13150 2550 30  0000 C CNN
 	1    13150 2450
@@
 $EndComp
 $Comp
-L -8V #PWR49
+L -8V #PWR51
 U 1 1 4B6DB78D
 P 13150 1400
-F 0 "#PWR49" H 13150 1530 20  0001 C CNN
+F 0 "#PWR51" H 13150 1530 20  0001 C CNN
 F 1 "3.3V" H 13150 1500 30  0000 C CNN
 	1    13150 1400
@@
 $EndComp
 $Comp
-L GND #PWR049
+L GND #PWR051
 U 1 1 4B6DB77B
 P 13150 2100
-F 0 "#PWR049" H 13150 2100 30  0001 C CNN
+F 0 "#PWR051" H 13150 2100 30  0001 C CNN
 F 1 "GND" H 13150 2030 30  0001 C CNN
 	1    13150 2100
@@
 TEST_MODE3
 $Comp
-L GND #PWR050
+L GND #PWR052
 U 1 1 4B6DB150
 P 2050 7550
-F 0 "#PWR050" H 2050 7550 30  0001 C CNN
+F 0 "#PWR052" H 2050 7550 30  0001 C CNN
 F 1 "GND" H 2050 7480 30  0001 C CNN
 	1    2050 7550
@@
 VCC3A3
 $Comp
-L -8V #PWR37
+L -8V #PWR39
 U 1 1 4B6DB004
 P 4650 1250
-F 0 "#PWR37" H 4650 1380 20  0001 C CNN
+F 0 "#PWR39" H 4650 1380 20  0001 C CNN
 F 1 "1V8D" H 4650 1350 30  0000 C CNN
 	1    4650 1250
@@
 $EndComp
 $Comp
-L -8V #PWR36
+L -8V #PWR38
 U 1 1 4B6DAFF8
 P 4050 1250
-F 0 "#PWR36" H 4050 1380 20  0001 C CNN
+F 0 "#PWR38" H 4050 1380 20  0001 C CNN
 F 1 "3.3V" H 4050 1350 30  0000 C CNN
 	1    4050 1250
@@
 $EndComp
 $Comp
-L -8V #PWR34
+L -8V #PWR36
 U 1 1 4B6DAFF2
 P 3750 1250
-F 0 "#PWR34" H 3750 1380 20  0001 C CNN
+F 0 "#PWR36" H 3750 1380 20  0001 C CNN
 F 1 "1V8A" H 3750 1350 30  0000 C CNN
 	1    3750 1250
@@
 $EndComp
 $Comp
-L -8V #PWR33
+L -8V #PWR35
 U 1 1 4B6DAFC6
 P 3550 1250
-F 0 "#PWR33" H 3550 1380 20  0001 C CNN
+F 0 "#PWR35" H 3550 1380 20  0001 C CNN
 F 1 "3V3A" H 3550 1350 30  0000 C CNN
 	1    3550 1250
@@
 $EndComp
 $Comp
-L GND #PWR051
+L GND #PWR053
 U 1 1 4B6DAEFD
 P 5200 7900
-F 0 "#PWR051" H 5200 7900 30  0001 C CNN
+F 0 "#PWR053" H 5200 7900 30  0001 C CNN
 F 1 "GND" H 5200 7830 30  0001 C CNN
 	1    5200 7900
@@
 $EndComp
 $Comp
-L GND #PWR052
+L GND #PWR054
 U 1 1 4B6DAEC0
 P 7100 2400
-F 0 "#PWR052" H 7100 2400 30  0001 C CNN
+F 0 "#PWR054" H 7100 2400 30  0001 C CNN
 F 1 "GND" H 7100 2330 30  0001 C CNN
 	1    7100 2400
@@
 $EndComp
 $Comp
-L GNDA #PWR053
+L GNDA #PWR055
 U 1 1 4B6DAEA9
 P 3800 7900
-F 0 "#PWR053" H 3800 7900 40  0001 C CNN
+F 0 "#PWR055" H 3800 7900 40  0001 C CNN
 F 1 "GNDA" H 3800 7830 40  0000 C CNN
 	1    3800 7900
