File: schematics/kicad_schematics/wiznet_network.sch (KiCad schematic (older format))
At the start: 49 parts, among them SW4 DIPS_03, U6 W5300, U7 RD1-125BAG1A, X4 25MHz

Commit message: modified pinout on em406, update schematic, and modified pinout on S08 and SSOT6
Parts:
- C23: footprint SM1210L -> 3v3_Tantulum_Capacitor
- C32, C34: footprint SM1210L -> 10uf_Tantulum_Capacitor
Changed lines of the file:
@@
-EESchema Schematic File Version 2  date Sun 14 Mar 2010 03:28:34 PM EDT
+EESchema Schematic File Version 2  date Sun 14 Mar 2010 03:55:01 PM EDT
 LIBS:power
 LIBS:device
@@
 NoConn ~ 2250 6700
 $Comp
-L GND #PWR038
+L GND #PWR037
 U 1 1 4B984217
 P 10950 7350
-F 0 "#PWR038" H 10950 7350 30  0001 C CNN
+F 0 "#PWR037" H 10950 7350 30  0001 C CNN
 F 1 "GND" H 10950 7280 30  0001 C CNN
 	1    10950 7350
@@
 A0 - GND IN 16-BIT MODE
 $Comp
-L GND #PWR039
+L GND #PWR038
 U 1 1 4B903065
 P 1400 5250
-F 0 "#PWR039" H 1400 5250 30  0001 C CNN
+F 0 "#PWR038" H 1400 5250 30  0001 C CNN
 F 1 "GND" H 1400 5180 30  0001 C CNN
 	1    1400 5250
@@
 $EndComp
 $Comp
-L GND #PWR040
+L GND #PWR039
 U 1 1 4B6DC2F1
 P 8350 9700
-F 0 "#PWR040" H 8350 9700 30  0001 C CNN
+F 0 "#PWR039" H 8350 9700 30  0001 C CNN
 F 1 "GND" H 8350 9630 30  0001 C CNN
 	1    8350 9700
@@
 $EndComp
 $Comp
-L GNDA #PWR041
+L GNDA #PWR040
 U 1 1 4B6DC0F8
 P 9450 4750
-F 0 "#PWR041" H 9450 4750 40  0001 C CNN
+F 0 "#PWR040" H 9450 4750 40  0001 C CNN
 F 1 "GNDA" H 9450 4680 40  0000 C CNN
 	1    9450 4750
@@
 $EndComp
 $Comp
-L GNDA #PWR042
+L GNDA #PWR041
 U 1 1 4B6DC0D3
 P 10150 7350
-F 0 "#PWR042" H 10150 7350 40  0001 C CNN
+F 0 "#PWR041" H 10150 7350 40  0001 C CNN
 F 1 "GNDA" H 10150 7280 40  0000 C CNN
 	1    10150 7350
@@
 $EndComp
 $Comp
-L GNDA #PWR043
+L GNDA #PWR042
 U 1 1 4B6DC05D
 P 9450 7450
-F 0 "#PWR043" H 9450 7450 40  0001 C CNN
+F 0 "#PWR042" H 9450 7450 40  0001 C CNN
 F 1 "GNDA" H 9450 7380 40  0000 C CNN
 	1    9450 7450
@@
 $EndComp
 $Comp
-L GND #PWR044
+L GND #PWR043
 U 1 1 4B6DB951
 P 13150 5650
-F 0 "#PWR044" H 13150 5650 30  0001 C CNN
+F 0 "#PWR043" H 13150 5650 30  0001 C CNN
 F 1 "GND" H 13150 5580 30  0001 C CNN
 	1    13150 5650
@@
 F 0 "C32" H 14450 5400 50  0000 L CNN
 F 1 "10uF/16V" H 14450 5200 50  0000 L CNN
-F 2 "SM1210L" H 14400 5300 60  0001 C CNN
+F 2 "10uf_Tantulum_Capacitor" H 14400 5300 60  0001 C CNN
 F 4 "Tant" H 14400 5300 60  0001 C CNN "TypeOfCap"
 	1    14400 5300
@@
 $EndComp
 $Comp
-L GNDA #PWR045
+L GNDA #PWR044
 U 1 1 4B6DB94B
 P 14400 5650
-F 0 "#PWR045" H 14400 5650 40  0001 C CNN
+F 0 "#PWR044" H 14400 5650 40  0001 C CNN
 F 1 "GNDA" H 14400 5580 40  0000 C CNN
 	1    14400 5650
@@
 1V8_OUT
 $Comp
-L GNDA #PWR046
+L GNDA #PWR045
 U 1 1 4B6DB901
 P 14400 4200
-F 0 "#PWR046" H 14400 4200 40  0001 C CNN
+F 0 "#PWR045" H 14400 4200 40  0001 C CNN
 F 1 "GNDA" H 14400 4130 40  0000 C CNN
 	1    14400 4200
@@
 F 0 "C34" H 14750 3950 50  0000 L CNN
 F 1 "10uF/16V" H 14750 3750 50  0000 L CNN
-F 2 "SM1210L" H 14700 3850 60  0001 C CNN
+F 2 "10uf_Tantulum_Capacitor" H 14700 3850 60  0001 C CNN
 F 4 "Tant" H 14700 3850 60  0001 C CNN "TypeOfCap"
 	1    14700 3850
@@
 $EndComp
 $Comp
-L GND #PWR047
+L GND #PWR046
 U 1 1 4B6DB886
 P 13150 4200
-F 0 "#PWR047" H 13150 4200 30  0001 C CNN
+F 0 "#PWR046" H 13150 4200 30  0001 C CNN
 F 1 "GND" H 13150 4130 30  0001 C CNN
 	1    13150 4200
@@
 F 0 "C23" H 13500 3950 50  0000 L CNN
 F 1 "3.3uF_Tant" H 13500 3750 50  0000 L CNN
-F 2 "SM1210L" H 13450 3850 60  0001 C CNN
+F 2 "3v3_Tantulum_Capacitor" H 13450 3850 60  0001 C CNN
 F 4 "Tant" H 13450 3850 60  0001 C CNN "TypeOfCap"
 	1    13450 3850
@@
 $EndComp
 $Comp
-L GNDA #PWR048
+L GNDA #PWR047
 U 1 1 4B6DB84F
 P 15850 1750
-F 0 "#PWR048" H 15850 1750 40  0001 C CNN
+F 0 "#PWR047" H 15850 1750 40  0001 C CNN
 F 1 "GNDA" H 15850 1680 40  0000 C CNN
 	1    15850 1750
@@
 $EndComp
 $Comp
-L GND #PWR049
+L GND #PWR048
 U 1 1 4B6DB842
 P 15250 1750
-F 0 "#PWR049" H 15250 1750 30  0001 C CNN
+F 0 "#PWR048" H 15250 1750 30  0001 C CNN
 F 1 "GND" H 15250 1680 30  0001 C CNN
 	1    15250 1750
@@
 $EndComp
 $Comp
-L GND #PWR050
+L GND #PWR049
 U 1 1 4B6DB7C7
 P 13150 3150
-F 0 "#PWR050" H 13150 3150 30  0001 C CNN
+F 0 "#PWR049" H 13150 3150 30  0001 C CNN
 F 1 "GND" H 13150 3080 30  0001 C CNN
 	1    13150 3150
@@
 $EndComp
 $Comp
-L GND #PWR051
+L GND #PWR050
 U 1 1 4B6DB77B
 P 13150 2100
-F 0 "#PWR051" H 13150 2100 30  0001 C CNN
+F 0 "#PWR050" H 13150 2100 30  0001 C CNN
 F 1 "GND" H 13150 2030 30  0001 C CNN
 	1    13150 2100
@@
 TEST_MODE3
 $Comp
-L GND #PWR052
+L GND #PWR051
 U 1 1 4B6DB150
 P 2050 7550
-F 0 "#PWR052" H 2050 7550 30  0001 C CNN
+F 0 "#PWR051" H 2050 7550 30  0001 C CNN
 F 1 "GND" H 2050 7480 30  0001 C CNN
 	1    2050 7550
@@
 $EndComp
 $Comp
-L GND #PWR053
+L GND #PWR052
 U 1 1 4B6DAEFD
 P 5200 7900
-F 0 "#PWR053" H 5200 7900 30  0001 C CNN
+F 0 "#PWR052" H 5200 7900 30  0001 C CNN
 F 1 "GND" H 5200 7830 30  0001 C CNN
 	1    5200 7900
@@
 $EndComp
 $Comp
-L GND #PWR054
+L GND #PWR053
 U 1 1 4B6DAEC0
 P 7100 2400
-F 0 "#PWR054" H 7100 2400 30  0001 C CNN
+F 0 "#PWR053" H 7100 2400 30  0001 C CNN
 F 1 "GND" H 7100 2330 30  0001 C CNN
 	1    7100 2400
@@
 $EndComp
 $Comp
-L GNDA #PWR055
+L GNDA #PWR054
 U 1 1 4B6DAEA9
 P 3800 7900
-F 0 "#PWR055" H 3800 7900 40  0001 C CNN
+F 0 "#PWR054" H 3800 7900 40  0001 C CNN
 F 1 "GNDA" H 3800 7830 40  0000 C CNN
 	1    3800 7900

Commit message: modified magjack
Parts:
- added R?: 0, SM0805, symbol R
Connections:
- wire segments 193 -> 194
Changed lines of the file:
@@
-EESchema Schematic File Version 2  date Sun 14 Mar 2010 03:55:01 PM EDT
+EESchema Schematic File Version 2  date Mon 15 Mar 2010 01:44:05 PM EDT
 LIBS:power
 LIBS:device
@@
 Sheet 4 5
 Title ""
-Date "14 mar 2010"
+Date "15 mar 2010"
 Rev ""
 Comp ""
@@
 Comment4 ""
 $EndDescr
-Wire Wire Line
-	11450 1800 10850 1800
+Connection ~ 10150 6100
+Wire Wire Line
+	10300 6100 10150 6100
+Wire Wire Line
+	10850 1800 11450 1800
 Connection ~ 13750 1950
 Connection ~ 13750 1550
@@
 Connection ~ 10150 5800
 Wire Wire Line
-	11100 5800 10150 5800
+	10150 5800 11100 5800
 Wire Notes Line
 	5250 8350 1100 8350
@@
 Connection ~ 9550 8800
 Wire Wire Line
-	8850 8800 10050 8800
+	10050 8800 8850 8800
 Connection ~ 9150 9600
 Wire Wire Line
@@
 	9300 5450 9300 5700
 Wire Wire Line
-	11100 6300 8450 6300
-Wire Wire Line
-	11100 5700 8450 5700
+	8450 6300 11100 6300
+Wire Wire Line
+	8450 5700 11100 5700
 Wire Wire Line
 	9600 4950 9600 4850
@@
 	11100 3050 11200 3050
 Wire Wire Line
-	11450 2750 11100 2750
+	11100 2750 11450 2750
 Wire Wire Line
 	10100 3050 9600 3050
@@
 Connection ~ 10950 1800
 Wire Wire Line
-	10950 1800 10950 1750
-Wire Wire Line
-	14200 3650 14700 3650
+	10950 1750 10950 1800
+Wire Wire Line
+	14700 3650 14200 3650
 Connection ~ 14400 3650
 Wire Wire Line
@@
 Connection ~ 4650 1550
 Wire Wire Line
-	4650 1250 4650 1650
+	4650 1650 4650 1250
 Connection ~ 4350 1550
 Wire Wire Line
@@
 	4150 1550 4150 1650
 Wire Wire Line
-	4050 1650 4050 1250
-Wire Wire Line
-	3750 1650 3750 1250
+	4050 1250 4050 1650
+Wire Wire Line
+	3750 1250 3750 1650
 Connection ~ 3900 7800
 Wire Wire Line
@@
 	4300 7800 4300 7700
 Wire Wire Line
-	5200 7900 5200 7700
+	5200 7700 5200 7900
 Wire Wire Line
 	5800 2150 6500 2150
@@
 	9600 7350 9600 7250
 Wire Wire Line
-	10150 6500 10150 4750
-Wire Wire Line
-	11100 5600 8450 5600
-Wire Wire Line
-	11100 6200 8450 6200
+	10150 4750 10150 6500
+Wire Wire Line
+	8450 5600 11100 5600
+Wire Wire Line
+	8450 6200 11100 6200
 Wire Wire Line
 	9600 5450 9600 5600
@@
 Connection ~ 9300 6200
 Wire Wire Line
-	9150 8900 9150 8800
+	9150 8800 9150 8900
 Wire Wire Line
 	8350 9600 8450 9600
@@
 	8450 8800 8350 8800
 Wire Wire Line
-	9550 8800 9550 8950
+	9550 8950 9550 8800
 Connection ~ 9150 8800
 Wire Wire Line
-	8850 9600 10050 9600
+	10050 9600 8850 9600
 Connection ~ 9550 9600
 Wire Wire Line
@@
 	1400 5100 1400 5250
 Wire Wire Line
-	11100 6100 10150 6100
-Connection ~ 10150 6100
-Wire Wire Line
-	13600 3650 12650 3650
+	12650 3650 13600 3650
 Connection ~ 13450 3650
 Connection ~ 13450 2600
@@
 Connection ~ 13450 1950
 Wire Wire Line
-	3800 7900 3800 7700
+	3800 7700 3800 7900
+Wire Wire Line
+	11100 6100 10800 6100
+$Comp
+L R R?
+U 1 1 4B9E7074
+P 10550 6100
+F 0 "R?" V 10630 6100 50  0000 C CNN
+F 1 "0" V 10550 6100 50  0000 C CNN
+F 2 "SM0805" H 10550 6100 60  0001 C CNN
+	1    10550 6100
+	0    -1   -1   0
+$EndComp
 $Comp
 L 1SS181 D19
@@
 U 1 1 4B6DC0FA
 P 9600 5200
-F 0 "R44" H 9500 5200 50  0000 C CNN
+F 0 "R44" V 9500 5200 50  0000 C CNN
 F 1 "49.9" V 9600 5200 50  0000 C CNN
 F 2 "SM0805" H 9600 5200 60  0001 C CNN
@@
 U 1 1 4B6DC0F9
 P 9300 5200
-F 0 "R41" H 9200 5200 50  0000 C CNN
+F 0 "R41" V 9200 5200 50  0000 C CNN
 F 1 "49.9" V 9300 5200 50  0000 C CNN
 F 2 "SM0805" H 9300 5200 60  0001 C CNN
@@
 U 1 1 4B6DBFA1
 P 10700 5200
-F 0 "R47" H 10600 5200 50  0000 C CNN
+F 0 "R47" V 10600 5200 50  0000 C CNN
 F 1 "200" V 10700 5200 50  0000 C CNN
 F 2 "SM0805" H 10700 5200 60  0001 C CNN
@@
 U 1 1 4B6DBFA0
 P 10400 5200
-F 0 "R46" H 10300 5200 50  0000 C CNN
+F 0 "R46" V 10300 5200 50  0000 C CNN
 F 1 "200" V 10400 5200 50  0000 C CNN
 F 2 "SM0805" H 10400 5200 60  0001 C CNN
@@
 U 1 1 4B6DBF70
 P 9300 7000
-F 0 "R42" H 9200 7000 50  0000 C CNN
+F 0 "R42" V 9200 7000 50  0000 C CNN
 F 1 "49.9" V 9300 7000 50  0000 C CNN
 F 2 "SM0805" H 9300 7000 60  0001 C CNN
@@
 U 1 1 4B6DBF56
 P 9600 7000
-F 0 "R45" H 9500 7000 50  0000 C CNN
+F 0 "R45" V 9500 7000 50  0000 C CNN
 F 1 "49.9" V 9600 7000 50  0000 C CNN
 F 2 "SM0805" H 9600 7000 60  0001 C CNN
