File: schematics/kicad_schematics/bearboard.orig.sch (KiCad schematic (older format))
At the start: 92 parts, among them P1 KOBICONN, P11 CONN_10X2, P2 CONN_10X2, P3 CONN_10X2, P4 CONN_10X2, P5 CONN_10X2, P6 CONN_10X2, P7 CONN_10X2, P8 CONN_10X2, P9 CONN_7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

Commit message: ran auto router and almost finalized
Parts:
- added P10: CONN_4, PIN_ARRAY_4x1, symbol CONN_4
- added R16: 4.7k, SM0805-CUSTOM, symbol R
- added R17: 2.6k, SM0805-CUSTOM, symbol R
- added U4: EMA406GPS, EM406, symbol EMA406GPS
Connections:
- net 5V0: now also U4.2 (VCC)
- net ADDR0: now also P7.1 (P1)
- net ADDR1: now also P7.2 (P2)
- net ADDR2: now also P7.3 (P3)
- net ADDR3: now also P7.4 (P4)
- net ADDR4: now also P7.5 (P5)
- net ADDR5: now also P7.6 (P6)
- net ADDR6: now also P7.13 (P13)
- net ADDR7: now also P7.14 (P14)
- net ADDR8: now also P7.15 (P15)
- net BT_RX: now also P10.2 (P2), R16.2, R17.2
- net BT_TX: now also P10.1 (P1), U4.3 (RX)
- net CTS: now also P10.4 (P4)
- net D0: now also P5.15 (P15)
- net D1: now also P5.16 (P16)
- net D10: now also P6.14 (P14)
- net D11: now also P6.15 (P15)
- net D12: now also P6.16 (P16)
- net D13: now also P5.9 (P9)
- net D14: now also P5.10 (P10)
- net D15: now also P5.11 (P11)
- net D2: now also P5.1 (P1)
- net D3: now also P5.2 (P2)
- net D4: now also P6.8 (P8)
- net D5: now also P6.9 (P9)
- net D6: now also P6.10 (P10)
- net D7: now also P6.11 (P11)
- net D8: now also P6.12 (P12)
- net D9: now also P6.13 (P13)
- net GND: now also R16.1, U4.1 (GND), U4.5 (GND)
- net PA1: now also P10.3 (P3)
- new net: R17.1, U4.4 (TX)
- no-connect marks 31 -> 7
Other:
- note added: "GPS CONNECTOR"
- note added: "Optional UART2 Connector"
